Commit message: 230725

File: dasom_description/urdf/try.urdf.xacro (robot description, xacro)
@@ -1,5 +1,13 @@
 <?xml version="1.0"?>
 <!-- Dasom Chain -->
-<robot name="dasom_try" xmlns:xacro="http://ros.org/wiki/xacro">
+<robot name="dasom_manipulator" xmlns:xacro="http://ros.org/wiki/xacro">
+  <xacro:property name="l1" value="0.034"/>
+  <xacro:property name="l2" value="0.05465"/>
+  <xacro:property name="l3" value="0.1585"/>
+  <xacro:property name="l4" value="0.099"/>
+  <xacro:property name="l5" value="0.04233"/>
+  <xacro:property name="l6" value="0.06975"/>
+  <xacro:property name="l7" value="0.04233"/>
+  <xacro:property name="l8" value="0.1"/>
   <!-- Import Rviz colors -->
   <xacro:include filename="$(find dasom_description)/urdf/materials.xacro" />
@@ -15,5 +23,5 @@
   <link name="link1">
     <visual>
-      <origin xyz="0 0 0" rpy="0 0 1.57"/>
+      <origin xyz="0 -0.012 ${-l1}" rpy="0 0 1.57"/>
       <geometry>
         <mesh filename="package://dasom_description/meshes/chain_link1.stl" scale="0.001 0.001 0.001"/>
@@ -36,8 +44,8 @@
   </link>
   <!-- Joint 1 -->
-  <joint name="joint1" type="revolute">
+  <joint name="id_1" type="revolute">
     <parent link="link1"/>
     <child link="link2"/>
-    <origin xyz="0.0 0.012 0.034" rpy="0 0 0"/>
+    <origin xyz="0 0 0" rpy="0 0 0"/>
     <axis xyz="0 0 1"/>
     <limit velocity="4.8" effort="1" lower="${-pi*0.9}" upper="${pi*0.9}" />
@@ -46,19 +54,19 @@
   <link name="link2">
     <visual>
-      <origin xyz="0 0 0.002" rpy="0 0 -1.57"/>
-      <geometry>
-        <mesh filename="package://dasom_description/meshes/chain_link2.stl" scale="0.001 0.001 0.001"/>
-      </geometry>
-      <material name="grey"/>
-    </visual>
-    <collision>
-      <origin xyz="0 0 0.002" rpy="0 0 0"/>
-      <geometry>
-        <mesh filename="package://dasom_description/meshes/chain_link2.stl" scale="0.001 0.001 0.001"/>
-      </geometry>
-    </collision>
-    <inertial>
-      <origin xyz="-3.0184870e-04 5.4043684e-04 ${0.018 + 2.9433464e-02}" />
-      <mass value="9.8406837e-02" />
+      <origin xyz="29.8e-03 -26e-03 0e-03" rpy="${pi*0.5} 0 ${pi}"/>
+      <geometry>
+        <mesh filename="package://dasom_description/meshes/Link1.STL.stl" scale="0.001 0.001 0.001"/>
+      </geometry>
+      <material name="grey"/>
+    </visual>
+    <collision>
+      <origin xyz="0 0 0" rpy="0 0 0"/>
+      <geometry>
+        <mesh filename="package://dasom_description/meshes/Link1.STL.stl" scale="0.001 0.001 0.001"/>
+      </geometry>
+    </collision>
+    <inertial>
+      <origin xyz="0.49e-03 0e-03 34.97e-03" />
+      <mass value="177.7e-03" />
       <inertia ixx="3.4543422e-05" ixy="-1.6031095e-08" ixz="-3.8375155e-07"
                iyy="3.2689329e-05" iyz="2.8511935e-08"
@@ -67,8 +75,8 @@
   </link>
   <!--  Joint 2 -->
-  <joint name="joint2" type="revolute">
+  <joint name="id_2" type="revolute">
     <parent link="link2"/>
     <child link="link3"/>
-    <origin xyz="0.0 0.0 0.0425" rpy="1.57 0 1.57"/>
+    <origin xyz="0.0 0.0 ${l2}" rpy="1.57 0 1.57"/>
     <axis xyz="0 0 1"/>
     <limit velocity="4.8" effort="1" lower="-0.15" upper="${pi}" />
@@ -77,19 +85,19 @@
   <link name="link3">
     <visual>
-      <origin xyz="0 0 0" rpy="1.57 0 1.57"/>
-      <geometry>
-        <mesh filename="package://dasom_description/meshes/chain_link3.stl" scale="0.001 0.001 0.001"/>
-      </geometry>
-      <material name="grey"/>
-    </visual>
-    <collision>
-      <origin xyz="0 0 0" rpy="0 0 0"/>
-      <geometry>
-        <mesh filename="package://dasom_description/meshes/chain_link3.stl" scale="0.001 0.001 0.001"/>
-      </geometry>
-    </collision>
-    <inertial>
-      <origin xyz="1.0308393e-02 3.7743363e-04 1.0170197e-01" />
-      <mass value="1.3850917e-01" />
+      <origin xyz="-15e-03 -17.5e-03 -28.5e-03" rpy="0 0 0"/>
+      <geometry>
+        <mesh filename="package://dasom_description/meshes/Link2.STL.stl" scale="0.001 0.001 0.001"/>
+      </geometry>
+      <material name="grey"/>
+    </visual>
+    <collision>
+      <origin xyz="0 0 0" rpy="0 0 0"/>
+      <geometry>
+        <mesh filename="package://dasom_description/meshes/Link2.STL.stl" scale="0.001 0.001 0.001"/>
+      </geometry>
+    </collision>
+    <inertial>
+      <origin xyz="-0.43e-03 128.84e-03 ${l2}" />
+      <mass value="201e-03" />
       <inertia ixx="3.3055381e-04" ixy="-9.7940978e-08" ixz="-3.8505711e-05"
                iyy="3.4290447e-04" iyz="-1.5717516e-06"
@@ -98,8 +106,8 @@
   </link>
   <!--  Joint 3 -->
-  <joint name="joint3" type="revolute">
+  <joint name="id_3" type="revolute">
     <parent link="link3"/>
     <child link="link4"/>
-    <origin xyz="0.128 0 0" rpy="0 0 0"/>
+    <origin xyz="${l3} 0 0" rpy="0 0 0"/>
     <axis xyz="0 0 1"/>
     <limit velocity="4.8" effort="1" lower="${-pi+0.4}" upper="${pi-0.4}" />
@@ -108,19 +116,19 @@
   <link name="link4">
     <visual>
-      <origin xyz="0 0 0" rpy="${pi/2} 0 0"/>
-      <geometry>
-        <mesh filename="package://dasom_description/meshes/chain_link4.stl" scale="0.001 0.001 0.001"/>
-      </geometry>
-      <material name="grey"/>
-    </visual>
-    <collision>
-      <origin xyz="0 0 0" rpy="0 0 0"/>
-      <geometry>
-        <mesh filename="package://dasom_description/meshes/chain_link4.stl" scale="0.001 0.001 0.001"/>
-      </geometry>
-    </collision>
-    <inertial>
-      <origin xyz="9.0909590e-02 3.8929816e-04 2.2413279e-04" />
-      <mass value="1.3274562e-01" />
+      <origin xyz="-15e-03 -15e-03 -28.5e-03" rpy="0 0 0"/>
+      <geometry>
+        <mesh filename="package://dasom_description/meshes/link3_ver2_3.STL.stl" scale="0.001 0.001 0.001"/>
+      </geometry>
+      <material name="grey"/>
+    </visual>
+    <collision>
+      <origin xyz="0 0 0" rpy="0 0 0"/>
+      <geometry>
+        <mesh filename="package://dasom_description/meshes/link3_ver2_3.STL.stl" scale="0.001 0.001 0.001"/>
+      </geometry>
+    </collision>
+    <inertial>
+      <origin xyz="0e-03 ${l3+60.16e-03} ${l2+1.84e-03}" />
+      <mass value="40e-03" />
       <inertia ixx="3.0654178e-05" ixy="-1.2764155e-06" ixz="-2.6874417e-07"
                iyy="2.4230292e-04" iyz="1.1559550e-08"
@@ -128,9 +136,9 @@
     </inertial>
   </link>
-   <!--  Joint 4 -->
-  <joint name="joint4" type="revolute">
+  <!--  Joint 4 -->
+  <joint name="id_4" type="revolute">
     <parent link="link4"/>
     <child link="link5"/>
-    <origin xyz="0.124 0.0 0.0" rpy="${pi*0.5} 0 ${pi*0.5}"/>
+    <origin xyz="${l4} 0.0 0.0" rpy="${pi*0.5} 0 ${pi*0.5}"/>
     <axis xyz="0 0 1"/>
     <limit velocity="4.8" effort="1" lower="${-pi*0.57}" upper="${pi*0.65}" />
@@ -139,14 +147,76 @@
   <link name="link5">
     <visual>
-      <origin xyz="0 0 0" rpy="0 0 0"/>
-      <geometry>
-        <mesh filename="package://dasom_description/meshes/chain_link5.stl" scale="0.001 0.001 0.001"/>
-      </geometry>
-      <material name="grey"/>
-    </visual>
-    <collision>
-      <origin xyz="0 0 0" rpy="0 0 0"/>
-      <geometry>
-        <mesh filename="package://dasom_description/meshes/chain_link5.stl" scale="0.001 0.001 0.001"/>
+      <origin xyz="-82.83e-03 -16.95e-03 81e-03" rpy="0 ${pi} ${-pi*0.5}"/>
+      <geometry>
+        <mesh filename="package://dasom_description/meshes/Link4.STL.stl" scale="0.001 0.001 0.001"/>
+      </geometry>
+      <material name="grey"/>
+    </visual>
+    <collision>
+      <origin xyz="0 0 0" rpy="0 0 0"/>
+      <geometry>
+        <mesh filename="package://dasom_description/meshes/Link4.STL.stl" scale="0.001 0.001 0.001"/>
+      </geometry>
+    </collision>
+    <inertial>
+      <origin xyz="0.36e-03 ${l3+l4+14.89e-03} ${l2-38.94e-03}" />
+      <mass value="186.70e-03" />
+      <inertia ixx="8.0870749e-05" ixy="0.0" ixz="-1.0157896e-06"
+               iyy="7.5980465e-05" iyz="0.0"
+               izz="9.3127351e-05" />
+    </inertial>
+  </link>
+  <!--  Joint 5 -->
+  <joint name="id_5" type="revolute">
+    <parent link="link5"/>
+    <child link="link6"/>
+    <origin xyz="${-l5} 0.0 ${l6}" rpy="${pi*0.5} 0 ${pi*0.5}"/>
+    <axis xyz="0 0 1"/>
+    <limit velocity="4.8" effort="1" lower="${-pi*0.57}" upper="${pi*0.65}" />
+  </joint>
+  <!--  Link 6 -->
+  <link name="link6">
+    <visual>
+      <origin xyz="-21e-03 -14.25e-03 -41.9e-03" rpy="0 0 0"/>
+      <geometry>
+        <mesh filename="package://dasom_description/meshes/Link5.STL.stl" scale="0.001 0.001 0.001"/>
+      </geometry>
+      <material name="grey"/>
+    </visual>
+    <collision>
+      <origin xyz="0 0 0" rpy="0 0 0"/>
+      <geometry>
+        <mesh filename="package://dasom_description/meshes/Link5.STL.stl" scale="0.001 0.001 0.001"/>
+      </geometry>
+    </collision>
+    <inertial>
+      <origin xyz="-1.98e-03 ${l3+l4+l6+0.67e-03} ${l2-l5+47.42e-03}" />
+      <mass value="94.3e-03"/>
+      <inertia ixx="8.0870749e-05" ixy="0.0" ixz="-1.0157896e-06"
+               iyy="7.5980465e-05" iyz="0.0"
+               izz="9.3127351e-05" />
+    </inertial>
+  </link>
+  <!--  Joint 6 -->
+  <joint name="id_6" type="revolute">
+    <parent link="link6"/>
+    <child link="link7"/>
+    <origin xyz="0 0 ${l7}" rpy="${pi*0.5} 0 ${pi*0.5}"/>
+    <axis xyz="0 0 1"/>
+    <limit velocity="4.8" effort="1" lower="${-pi*0.57}" upper="${pi*0.65}" />
+  </joint>
+  <!--  Link 7 -->
+  <link name="link7">
+    <visual>
+      <origin xyz="0 0 0" rpy="${pi*0.5} 0 0"/>
+      <geometry>
+        <mesh filename="package://dasom_description/meshes/chain_link4.stl" scale="0.001 0.001 0.001"/>
+      </geometry>
+      <material name="grey"/>
+    </visual>
+    <collision>
+      <origin xyz="0 0 0" rpy="0 0 0"/>
+      <geometry>
+        <mesh filename="package://dasom_description/meshes/chain_link4.stl" scale="0.001 0.001 0.001"/>
       </geometry>
     </collision>
@@ -159,3 +229,34 @@
     </inertial>
   </link>
+  <!--  Joint 7 -->
+  <joint name="id_7" type="fixed">
+    <parent link="link7"/>
+    <child link="link8"/>
+    <origin xyz="${l8} 0 0" rpy="${pi*0.5} 0 ${pi*0.5}"/>
+    <axis xyz="0 0 1"/>
+    <limit velocity="4.8" effort="1" lower="${-pi*0.5}" upper="${pi*0.5}" />
+  </joint>
+  <!--  Link 8 -->
+  <link name="link8">
+    <visual>
+      <origin xyz="0 0 0" rpy="0 ${-pi*0.5} 0"/>
+      <geometry>
+        <mesh filename="package://dasom_description/meshes/chain_link_grip_l.stl" scale="0.001 0.001 0.001"/>
+      </geometry>
+      <material name="grey"/>
+    </visual>
+    <collision>
+      <origin xyz="0 0 0" rpy="0 0 0"/>
+      <geometry>
+        <mesh filename="package://dasom_description/meshes/chain_link_grip_l.stl" scale="0.001 0.001 0.001"/>
+      </geometry>
+    </collision>
+    <inertial>
+      <origin xyz="4.4206755e-02 3.6839985e-07 8.9142216e-03" />
+      <mass value="1.4327573e-01" />
+      <inertia ixx="8.0870749e-05" ixy="0.0" ixz="-1.0157896e-06"
+               iyy="7.5980465e-05" iyz="0.0"
+               izz="9.3127351e-05" />
+    </inertial>
+  </link>
 </robot>

Commit message: 230727

File: dasom_description/urdf/try.urdf.xacro (robot description, xacro)
@@ -49,5 +49,5 @@
     <origin xyz="0 0 0" rpy="0 0 0"/>
     <axis xyz="0 0 1"/>
-    <limit velocity="4.8" effort="1" lower="${-pi*0.9}" upper="${pi*0.9}" />
+    <limit velocity="4.8" effort="1" lower="${-pi}" upper="${pi}" />
   </joint>
   <!--  Link 2 -->
@@ -80,5 +80,5 @@
     <origin xyz="0.0 0.0 ${l2}" rpy="1.57 0 1.57"/>
     <axis xyz="0 0 1"/>
-    <limit velocity="4.8" effort="1" lower="-0.15" upper="${pi}" />
+    <limit velocity="4.8" effort="1" lower="${-pi}" upper="${pi}" />
   </joint>
   <!--  Link 3 -->
@@ -111,5 +111,5 @@
     <origin xyz="${l3} 0 0" rpy="0 0 0"/>
     <axis xyz="0 0 1"/>
-    <limit velocity="4.8" effort="1" lower="${-pi+0.4}" upper="${pi-0.4}" />
+    <limit velocity="4.8" effort="1" lower="${-pi}" upper="${pi}" />
   </joint>
   <!--  Link 4 -->
@@ -142,5 +142,5 @@
     <origin xyz="${l4} 0.0 0.0" rpy="${pi*0.5} 0 ${pi*0.5}"/>
     <axis xyz="0 0 1"/>
-    <limit velocity="4.8" effort="1" lower="${-pi*0.57}" upper="${pi*0.65}" />
+    <limit velocity="4.8" effort="1" lower="${-pi}" upper="${pi}" />
   </joint>
   <!--  Link 5 -->

Commit message: 230802

File: dasom_description/urdf/try.urdf.xacro (robot description, xacro)
@@ -173,5 +173,5 @@
     <origin xyz="${-l5} 0.0 ${l6}" rpy="${pi*0.5} 0 ${pi*0.5}"/>
     <axis xyz="0 0 1"/>
-    <limit velocity="4.8" effort="1" lower="${-pi*0.57}" upper="${pi*0.65}" />
+    <limit velocity="4.8" effort="1" lower="${-pi}" upper="${pi}" />
   </joint>
   <!--  Link 6 -->
@@ -204,5 +204,5 @@
     <origin xyz="0 0 ${l7}" rpy="${pi*0.5} 0 ${pi*0.5}"/>
     <axis xyz="0 0 1"/>
-    <limit velocity="4.8" effort="1" lower="${-pi*0.57}" upper="${pi*0.65}" />
+    <limit velocity="4.8" effort="1" lower="${-pi}" upper="${pi}" />
   </joint>
   <!--  Link 7 -->
@@ -235,5 +235,5 @@
     <origin xyz="${l8} 0 0" rpy="${pi*0.5} 0 ${pi*0.5}"/>
     <axis xyz="0 0 1"/>
-    <limit velocity="4.8" effort="1" lower="${-pi*0.5}" upper="${pi*0.5}" />
+    <limit velocity="4.8" effort="1" lower="${-pi}" upper="${pi}" />
   </joint>
   <!--  Link 8 -->
