Commit message: 230810

File: dasom_description/urdf/dasom_paletrone.urdf.xacro (robot description, xacro)
@@ -23,4 +23,31 @@
   <joint name="base_joint_Z" type="prismatic">
     <parent link="base_link_Y"/>
+    <child link="base_link_Z" />
+    <origin xyz="0 0 0" rpy="0 0 0"/>
+    <axis xyz="0 0 1"/>
+    <limit lower="-0.5" upper="0.5" effort="100" velocity="0.1"/>
+  </joint>
+  <link name="base_link_Z"/>
+  <!-- Define Z-axis prismatic joint and link -->
+  <joint name="base_joint_r" type="revolute">
+    <parent link="base_link_Z"/>
+    <child link="base_link_r" />
+    <origin xyz="0 0 0" rpy="0 0 0"/>
+    <axis xyz="1 0 0"/>
+    <limit lower="-0.5" upper="0.5" effort="100" velocity="0.1"/>
+  </joint>
+  <link name="base_link_r"/>
+  <!-- Define Z-axis prismatic joint and link -->
+  <joint name="base_joint_p" type="revolute">
+    <parent link="base_link_r"/>
+    <child link="base_link_p" />
+    <origin xyz="0 0 0" rpy="0 0 0"/>
+    <axis xyz="0 1 0"/>
+    <limit lower="-0.5" upper="0.5" effort="100" velocity="0.1"/>
+  </joint>
+  <link name="base_link_p"/>
+  <!-- Define Z-axis prismatic joint and link -->
+  <joint name="base_joint_y" type="revolute">
+    <parent link="base_link_p"/>
     <child link="base_link" />
     <origin xyz="0 0 0" rpy="0 0 0"/>

Commit message: 230815

File: dasom_description/urdf/dasom_paletrone.urdf.xacro (robot description, xacro)
@@ -30,28 +30,28 @@
   <link name="base_link_Z"/>
   <!-- Define Z-axis prismatic joint and link -->
-  <joint name="base_joint_r" type="revolute">
+  <joint name="base_joint_y" type="revolute">
     <parent link="base_link_Z"/>
-    <child link="base_link_r" />
+    <child link="base_link_y" />
     <origin xyz="0 0 0" rpy="0 0 0"/>
-    <axis xyz="1 0 0"/>
-    <limit lower="-0.5" upper="0.5" effort="100" velocity="0.1"/>
+    <axis xyz="0 0 1"/>
+    <limit lower="-5" upper="5" effort="100" velocity="0.1"/>
   </joint>
-  <link name="base_link_r"/>
+  <link name="base_link_y"/>
   <!-- Define Z-axis prismatic joint and link -->
   <joint name="base_joint_p" type="revolute">
-    <parent link="base_link_r"/>
+    <parent link="base_link_y"/>
     <child link="base_link_p" />
     <origin xyz="0 0 0" rpy="0 0 0"/>
     <axis xyz="0 1 0"/>
-    <limit lower="-0.5" upper="0.5" effort="100" velocity="0.1"/>
+    <limit lower="-5" upper="5" effort="100" velocity="0.1"/>
   </joint>
   <link name="base_link_p"/>
   <!-- Define Z-axis prismatic joint and link -->
-  <joint name="base_joint_y" type="revolute">
+  <joint name="base_joint_r" type="revolute">
     <parent link="base_link_p"/>
     <child link="base_link" />
     <origin xyz="0 0 0" rpy="0 0 0"/>
-    <axis xyz="0 0 1"/>
-    <limit lower="-0.5" upper="0.5" effort="100" velocity="0.1"/>
+    <axis xyz="1 0 0"/>
+    <limit lower="-5" upper="5" effort="100" velocity="0.1"/>
   </joint>
   <link name="base_link">

Commit message: 230906

File: dasom_description/urdf/dasom_paletrone.urdf.xacro (robot description, xacro)
@@ -6,5 +6,5 @@
     <parent link="world"/>
     <child link="base_link_X" />
-    <origin xyz="0 0 0" rpy="0 0 0"/>
+    <origin xyz="-0.083278 0 0" rpy="0 0 0"/>
     <axis xyz="1 0 0"/>
     <limit lower="-0.5" upper="0.5" effort="100" velocity="0.1"/>
@@ -15,5 +15,5 @@
     <parent link="base_link_X"/>
     <child link="base_link_Y" />
-    <origin xyz="0 0 0" rpy="0 0 0"/>
+    <origin xyz="0 -0.053549 0" rpy="0 0 0"/>
     <axis xyz="0 1 0"/>
     <limit lower="-0.5" upper="0.5" effort="100" velocity="0.1"/>
@@ -24,5 +24,5 @@
     <parent link="base_link_Y"/>
     <child link="base_link_Z" />
-    <origin xyz="0 0 0" rpy="0 0 0"/>
+    <origin xyz="0 0 -0.001452" rpy="0 0 0"/>
     <axis xyz="0 0 1"/>
     <limit lower="-0.5" upper="0.5" effort="100" velocity="0.1"/>
@@ -33,5 +33,5 @@
     <parent link="base_link_Z"/>
     <child link="base_link_y" />
-    <origin xyz="0 0 0" rpy="0 0 0"/>
+    <origin xyz="0 0 0" rpy="0 0 ${-0.560295}"/>
     <axis xyz="0 0 1"/>
     <limit lower="-5" upper="5" effort="100" velocity="0.1"/>
@@ -42,5 +42,5 @@
     <parent link="base_link_y"/>
     <child link="base_link_p" />
-    <origin xyz="0 0 0" rpy="0 0 0"/>
+    <origin xyz="0 0 0" rpy="0 ${-1.558368} 0"/>
     <axis xyz="0 1 0"/>
     <limit lower="-5" upper="5" effort="100" velocity="0.1"/>
@@ -51,5 +51,5 @@
     <parent link="base_link_p"/>
     <child link="base_link" />
-    <origin xyz="0 0 0" rpy="0 0 0"/>
+    <origin xyz="0 0 0" rpy="${-1.035882} 0 0"/>
     <axis xyz="1 0 0"/>
     <limit lower="-5" upper="5" effort="100" velocity="0.1"/>

Commit message: 230913

File: dasom_description/urdf/dasom_paletrone.urdf.xacro (robot description, xacro)
@@ -6,5 +6,5 @@
     <parent link="world"/>
     <child link="base_link_X" />
-    <origin xyz="-0.083278 0 0" rpy="0 0 0"/>
+    <origin xyz="0 0 0" rpy="0 0 0"/>
     <axis xyz="1 0 0"/>
     <limit lower="-0.5" upper="0.5" effort="100" velocity="0.1"/>
@@ -15,5 +15,5 @@
     <parent link="base_link_X"/>
     <child link="base_link_Y" />
-    <origin xyz="0 -0.053549 0" rpy="0 0 0"/>
+    <origin xyz="0 0 0" rpy="0 0 0"/>
     <axis xyz="0 1 0"/>
     <limit lower="-0.5" upper="0.5" effort="100" velocity="0.1"/>
@@ -24,5 +24,5 @@
     <parent link="base_link_Y"/>
     <child link="base_link_Z" />
-    <origin xyz="0 0 -0.001452" rpy="0 0 0"/>
+    <origin xyz="0 0 0" rpy="0 0 0"/>
     <axis xyz="0 0 1"/>
     <limit lower="-0.5" upper="0.5" effort="100" velocity="0.1"/>
@@ -33,5 +33,5 @@
     <parent link="base_link_Z"/>
     <child link="base_link_y" />
-    <origin xyz="0 0 0" rpy="0 0 ${-0.560295}"/>
+    <origin xyz="0 0 0" rpy="0 0 0"/>
     <axis xyz="0 0 1"/>
     <limit lower="-5" upper="5" effort="100" velocity="0.1"/>
@@ -42,5 +42,5 @@
     <parent link="base_link_y"/>
     <child link="base_link_p" />
-    <origin xyz="0 0 0" rpy="0 ${-1.558368} 0"/>
+    <origin xyz="0 0 0" rpy="0 0 0"/>
     <axis xyz="0 1 0"/>
     <limit lower="-5" upper="5" effort="100" velocity="0.1"/>
@@ -51,5 +51,5 @@
     <parent link="base_link_p"/>
     <child link="base_link" />
-    <origin xyz="0 0 0" rpy="${-1.035882} 0 0"/>
+    <origin xyz="0 0 0" rpy="0 0 0"/>
     <axis xyz="1 0 0"/>
     <limit lower="-5" upper="5" effort="100" velocity="0.1"/>
